Commit message: Basis URDF

File: Assets/adt_urdf/basis_roboter_urdf/BasisRoboter.urdf (robot description, URDF)
Before this commit: robot BasisRoboter, 3 links, 2 joints
Links:
- link base_plate: geometry visual mesh filename=file:///urdf/basis_roboter_urdf/meshes/Solid1.stl scale=1 1 1
- link x: geometry visual mesh filename=file:///urdf/basis_roboter_urdf/meshes/MeshFeature1_10.stl scale=1 1 1; visual mesh filename=file:///urdf/basis_roboter_urdf/meshes/MeshFeature1_5.stl scale=1 1 1

Commit message: Basis URDF

File: Assets/adt_urdf/basis_roboter_urdf/BasisRoboter.urdf (robot description, URDF)
Before this commit: robot BasisRoboter, 3 links, 2 joints
Links:
- removed link base_plate
- added link y, mass 1; visual box size=0.05 0.2 0.05; visual box size=0.05 0.2 0.05
- added link z, mass 1; visual box size=0.15 0.25 0.025
- link base_link: geometry visual box size=0.1 0.6 0.025; visual box size=0.4 0.6 0.025
- link x: geometry visual box size=0.015 0.32 0.23; visual box size=0.015 0.32 0.23
Joints:
- removed joint base_link_base_plate_joint
- removed joint base_plate_x_joint
- added joint base_link_x_joint: type prismatic, parent base_link, child x, origin xyz=-0.5545 1.1553 0.0125, limit lower=0 upper=1.5 effort=3.40282346638529E+38 velocity=100
- added joint x_y_joint: type prismatic, parent x, child y, limit lower=0 upper=0 effort=3.40282346638529E+38 velocity=100
- added joint y_z_joint: type prismatic, parent y, child z, limit lower=0 upper=0 effort=3.40282346638529E+38 velocity=100

Commit message: BasisRoboter URDF Fix

File: Assets/adt_urdf/basis_roboter_urdf/BasisRoboter.urdf (robot description, URDF)
Before this commit: robot BasisRoboter, 4 links, 3 joints
Links:
- added link x_visu, mass 1; visual box size=0.015 0.32 0.23; visual box size=0.015 0.32 0.23
- added link y_visu, mass 1; visual box size=0.05 0.2 0.05; visual box size=0.05 0.2 0.05
- added link z_visu, mass 1; visual box size=0.15 0.25 0.025
- link x: geometry 
- link y: geometry 
- link z: geometry 
Joints:
- added joint x_x_visu_joint: type fixed, parent x, child x_visu, origin rpy=0 0 -4.712389
- added joint y_y_visu_joint: type fixed, parent y, child y_visu, origin rpy=-4.712389 0 -4.712389
- added joint z_z_visu_joint: type fixed, parent z, child z_visu, origin rpy=-4.712389 0 0
- joint base_link_x_joint: origin xyz=-0.5545 1.1553 0.0125 -> xyz=-0.5545 1.1553 0.0125 rpy=0 0 -1.570796
- joint x_y_joint: origin (none) -> rpy=0 4.712389 0
- joint y_z_joint: origin (none) -> rpy=0 0 -4.712389
