Commit message: Wheel Sim

File: Assets/adt_urdf/service_roboter_urdf/ServiceRoboter.urdf (robot description, URDF)
Before this commit: robot ServiceRoboter, 12 links, 12 joints
Links:
- added link sensor_front_1, mass 1; visual box size=0.03 0.03 0.03
- added link sensor_front_2, mass 1; visual box size=0.03 0.03 0.03
- added link sensor_front_3, mass 1; visual box size=0.03 0.03 0.03
- added link sensor_left_1, mass 1; visual box size=0.03 0.03 0.03
- added link sensor_left_2, mass 1; visual box size=0.03 0.03 0.03
- added link sensor_left_3, mass 1; visual box size=0.03 0.03 0.03
- added link sensor_right_1, mass 1; visual box size=0.03 0.03 0.03
- added link sensor_right_2, mass 1; visual box size=0.03 0.03 0.03
- added link sensor_right_3, mass 1; visual box size=0.03 0.03 0.03
- added link uss_base, mass 1
- added link uss_front, mass 1
- added link uss_left, mass 1
- added link uss_right, mass 1
- link lidar: geometry collision cylinder length=0.04 radius=0.05; visual cylinder length=0.04 radius=0.05
Joints:
- removed joint ServiceRoboter_base_link_joint
- added joint barrel_uss_base_joint: type fixed, parent barrel, child uss_base, origin xyz=0 0 0.8
- added joint front_sensor_1_joint: type fixed, parent uss_front, child sensor_front_1, origin xyz=0.28 0 0
- added joint front_sensor_2_joint: type fixed, parent uss_front, child sensor_front_2, origin xyz=0.28 0 -0.3
- added joint front_sensor_3_joint: type fixed, parent uss_front, child sensor_front_3, origin xyz=0.28 0 -0.6
- added joint left_sensor_1_joint: type fixed, parent uss_left, child sensor_left_1, origin xyz=0.28 0 0
- added joint left_sensor_2_joint: type fixed, parent uss_left, child sensor_left_2, origin xyz=0.28 0 -0.3
- added joint left_sensor_3_joint: type fixed, parent uss_left, child sensor_left_3, origin xyz=0.28 0 -0.6
- added joint right_sensor_1_joint: type fixed, parent uss_right, child sensor_right_1
- added joint right_sensor_2_joint: type fixed, parent uss_right, child sensor_right_2, origin xyz=0.28 0 -0.3
- added joint right_sensor_3_joint: type fixed, parent uss_right, child sensor_right_3, origin xyz=0.28 0 -0.6
- added joint uss_base_front_joint: type fixed, parent uss_base, child uss_front
- added joint uss_base_left_joint: type fixed, parent uss_base, child uss_left, origin rpy=0 0 -5.934119
- added joint uss_base_right_joint: type fixed, parent uss_base, child uss_right, origin rpy=0 0 -0.349066
- joint wheel_left_axis_wheel_left_joint: axis 1 0 0 -> (none)
- joint wheel_right_axis_wheel_right_joint: axis 1 0 0 -> (none)

Commit message: SLAM not working...

File: Assets/adt_urdf/service_roboter_urdf/ServiceRoboter.urdf (robot description, URDF)
Before this commit: robot ServiceRoboter, 25 links, 24 joints
Links:
- added link base_footprint, mass 1
Joints:
- removed joint front_sensor_1_joint
- removed joint front_sensor_2_joint
- removed joint front_sensor_3_joint
- removed joint left_sensor_1_joint
- removed joint left_sensor_2_joint
- removed joint left_sensor_3_joint
- removed joint right_sensor_1_joint
- removed joint right_sensor_2_joint
- removed joint right_sensor_3_joint
- removed joint uss_base_front_joint
- removed joint uss_base_left_joint
- removed joint uss_base_right_joint
- added joint base_link_base_footprint_joint: type fixed, parent base_link, child base_footprint
- added joint uss_base_uss_front_joint: type fixed, parent uss_base, child uss_front
- added joint uss_base_uss_left_joint: type fixed, parent uss_base, child uss_left, origin rpy=0 0 -5.934119
- added joint uss_base_uss_right_joint: type fixed, parent uss_base, child uss_right, origin rpy=0 0 -0.349066
- added joint uss_front_sensor_front_1_joint: type fixed, parent uss_front, child sensor_front_1, origin xyz=0.28 0 0
- added joint uss_front_sensor_front_2_joint: type fixed, parent uss_front, child sensor_front_2, origin xyz=0.28 0 -0.3
- added joint uss_front_sensor_front_3_joint: type fixed, parent uss_front, child sensor_front_3, origin xyz=0.28 0 -0.6
- added joint uss_left_sensor_left_1_joint: type fixed, parent uss_left, child sensor_left_1, origin xyz=0.28 0 0
- added joint uss_left_sensor_left_2_joint: type fixed, parent uss_left, child sensor_left_2, origin xyz=0.28 0 -0.3
- added joint uss_left_sensor_left_3_joint: type fixed, parent uss_left, child sensor_left_3, origin xyz=0.28 0 -0.6
- added joint uss_right_sensor_right_1_joint: type fixed, parent uss_right, child sensor_right_1
- added joint uss_right_sensor_right_2_joint: type fixed, parent uss_right, child sensor_right_2, origin xyz=0.28 0 -0.3
- added joint uss_right_sensor_right_3_joint: type fixed, parent uss_right, child sensor_right_3, origin xyz=0.28 0 -0.6
- joint wheel_base_wheel_back_axis_joint: origin xyz=0 0 -0.04 -> xyz=0 0 -0.045
- joint wheel_base_wheel_front_axis_joint: origin xyz=0.2 0 -0.04 -> xyz=0.2 0 -0.045

File: Assets/adt_urdf/service_roboter_urdf/_backup/ServiceRoboter.urdf (robot description, URDF)
Before this commit: robot ServiceRoboter, 12 links, 11 joints
Links:
- added link sensor_front_1, mass 1; visual box size=0.03 0.03 0.03
- added link sensor_front_2, mass 1; visual box size=0.03 0.03 0.03
- added link sensor_front_3, mass 1; visual box size=0.03 0.03 0.03
- added link sensor_left_1, mass 1; visual box size=0.03 0.03 0.03
- added link sensor_left_2, mass 1; visual box size=0.03 0.03 0.03
- added link sensor_left_3, mass 1; visual box size=0.03 0.03 0.03
- added link sensor_right_1, mass 1; visual box size=0.03 0.03 0.03
- added link sensor_right_2, mass 1; visual box size=0.03 0.03 0.03
- added link sensor_right_3, mass 1; visual box size=0.03 0.03 0.03
- added link uss_base, mass 1
- added link uss_front, mass 1
- added link uss_left, mass 1
- added link uss_right, mass 1
- link lidar: geometry collision cylinder length=0.04 radius=0.05; visual cylinder length=0.04 radius=0.05
Joints:
- added joint barrel_uss_base_joint: type fixed, parent barrel, child uss_base, origin xyz=0 0 0.8
- added joint front_sensor_1_joint: type fixed, parent uss_front, child sensor_front_1, origin xyz=0.28 0 0
- added joint front_sensor_2_joint: type fixed, parent uss_front, child sensor_front_2, origin xyz=0.28 0 -0.3
- added joint front_sensor_3_joint: type fixed, parent uss_front, child sensor_front_3, origin xyz=0.28 0 -0.6
- added joint left_sensor_1_joint: type fixed, parent uss_left, child sensor_left_1, origin xyz=0.28 0 0
- added joint left_sensor_2_joint: type fixed, parent uss_left, child sensor_left_2, origin xyz=0.28 0 -0.3
- added joint left_sensor_3_joint: type fixed, parent uss_left, child sensor_left_3, origin xyz=0.28 0 -0.6
- added joint right_sensor_1_joint: type fixed, parent uss_right, child sensor_right_1
- added joint right_sensor_2_joint: type fixed, parent uss_right, child sensor_right_2, origin xyz=0.28 0 -0.3
- added joint right_sensor_3_joint: type fixed, parent uss_right, child sensor_right_3, origin xyz=0.28 0 -0.6
- added joint uss_base_front_joint: type fixed, parent uss_base, child uss_front
- added joint uss_base_left_joint: type fixed, parent uss_base, child uss_left, origin rpy=0 0 -5.934119
- added joint uss_base_right_joint: type fixed, parent uss_base, child uss_right, origin rpy=0 0 -0.349066
- joint wheel_base_wheel_back_axis_joint: origin xyz=0 0 0.01 -> xyz=0 0 -0.04
- joint wheel_base_wheel_front_axis_joint: origin xyz=0.2 0 0.01 -> xyz=0.2 0 -0.04
